Commit message: fix: fix relative angles

File: generated/robot.urdf (robot description, URDF)
Before this commit: robot pydantic_robot, 15 links, 14 joints
Links:
- link base: geometry collision box size=0.08 0.08 0.02; visual box size=0.08 0.08 0.02
Joints:
- joint j_base_to_f2_s1: origin xyz=0.05083530666080496 0.031871171875253006 0.01 rpy=0 0 0.56 -> xyz=0.05083530666080497 0.031871171875253 0.01 rpy=0 0 0.5599999999999998
- joint j_base_to_f3_s1: origin xyz=0.059135086014573644 0.01015094094401976 0.01 rpy=0 0 0.17 -> xyz=0.059135086014573644 0.01015094094401975 0.01 rpy=0 0 0.16999999999999982
- joint j_base_to_f4_s1: origin xyz=0.058803994670474494 -0.011920159847703672 0.01 rpy=0 0 -0.2 -> xyz=0.058803994670474494 -0.011920159847703683 0.01 rpy=0 0 -0.20000000000000018
- joint j_base_to_f5_s1: origin xyz=0.058529061652924 -0.028272759717229968 0.01 rpy=0 0 -0.45 -> xyz=0.058529061652924 -0.028272759717229975 0.01 rpy=0 0 -0.4500000000000002

Commit message: chore: remove 2d simulation

File: generated/robot.urdf (robot description, URDF)
Before this commit: robot pydantic_robot, 15 links, 14 joints
Links:
- removed link f5_s1
- removed link f5_s2
- removed link f5_s3
- added link f1_s3, mass 0.02; collision cylinder length=0.03 radius=0.008; visual cylinder length=0.03 radius=0.008
- link base: mass 0.4 -> 0.5; geometry collision box size=0.1 0.1 0.02; visual box size=0.1 0.1 0.02
- link f1_s1: mass 0.06 -> 0.05; geometry collision cylinder length=0.05 radius=0.01; visual cylinder length=0.05 radius=0.01
- link f1_s2: mass 0.05 -> 0.03; geometry collision cylinder length=0.04 radius=0.009; visual cylinder length=0.04 radius=0.009
- link f2_s1: mass 0.045 -> 0.05; geometry collision cylinder length=0.05 radius=0.01; visual cylinder length=0.05 radius=0.01
- link f2_s2: mass 0.035 -> 0.03; geometry collision cylinder length=0.04 radius=0.009; visual cylinder length=0.04 radius=0.009
- link f2_s3: mass 0.025 -> 0.02; geometry collision cylinder length=0.03 radius=0.008; visual cylinder length=0.03 radius=0.008
- link f3_s1: geometry collision cylinder length=0.05 radius=0.01; visual cylinder length=0.05 radius=0.01
- link f3_s2: mass 0.04 -> 0.03
- link f3_s3: mass 0.025 -> 0.02; geometry collision cylinder length=0.03 radius=0.008; visual cylinder length=0.03 radius=0.008
- link f4_s1: mass 0.045 -> 0.05; geometry collision cylinder length=0.05 radius=0.01; visual cylinder length=0.05 radius=0.01
- link f4_s2: mass 0.035 -> 0.03; geometry collision cylinder length=0.04 radius=0.009; visual cylinder length=0.04 radius=0.009
- link f4_s3: mass 0.025 -> 0.02; geometry collision cylinder length=0.03 radius=0.008; visual cylinder length=0.03 radius=0.008
Joints:
- removed joint j_base_to_f5_s1
- removed joint j_f5_s1_to_f5_s2
- removed joint j_f5_s2_to_f5_s3
- added joint j_f1_s2_to_f1_s3: type revolute, parent f1_s2, child f1_s3, origin xyz=0 0 0.04 rpy=0 0 0, axis 0 1 0, limit lower=-0.7 upper=1.57 effort=10 velocity=1.0
- joint j_base_to_f1_s1: limit lower=-0.5 upper=1.2 effort=10 velocity=1.0 -> lower=-0.7 upper=1.57 effort=10 velocity=1.0; origin xyz=-0.024809445635299944 0.043410729172280636 0.01 rpy=0 0 2.96 -> xyz=0.05 0.0 0.0 rpy=0 0 3.1415
- joint j_base_to_f2_s1: limit lower=-0.3 upper=1.4 effort=10 velocity=1.0 -> lower=-0.7 upper=1.57 effort=10 velocity=1.0; origin xyz=0.05083530666080497 0.031871171875253 0.01 rpy=0 0 0.5599999999999998 -> xyz=3.981633553666317e-05 0.049999984146591736 0.0 rpy=0 0 4.7115
- joint j_base_to_f3_s1: limit lower=-0.3 upper=1.4 effort=10 velocity=1.0 -> lower=-0.7 upper=1.57 effort=10 velocity=1.0; origin xyz=0.059135086014573644 0.01015094094401975 0.01 rpy=0 0 0.16999999999999982 -> xyz=-0.00011944890561407693 -0.0499998573193859 0.0 rpy=0 0 7.8515
- joint j_base_to_f4_s1: limit lower=-0.3 upper=1.4 effort=10 velocity=1.0 -> lower=-0.7 upper=1.57 effort=10 velocity=1.0; origin xyz=0.058803994670474494 -0.011920159847703683 0.01 rpy=0 0 -0.20000000000000018 -> xyz=-0.049999429278357904 0.0002388971295064256 0.0 rpy=0 0 12.5615
- joint j_f1_s1_to_f1_s2: limit lower=-0.5 upper=1.2 effort=10 velocity=1.0 -> lower=-0.7 upper=1.57 effort=10 velocity=1.0; origin xyz=0 0 0.035 rpy=0 0 0 -> xyz=0 0 0.05 rpy=0 0 0
- joint j_f2_s1_to_f2_s2: limit lower=-0.3 upper=1.4 effort=10 velocity=1.0 -> lower=-0.7 upper=1.57 effort=10 velocity=1.0; origin xyz=0 0 0.055 rpy=0 0 0 -> xyz=0 0 0.05 rpy=0 0 0
- joint j_f2_s2_to_f2_s3: limit lower=-0.3 upper=1.4 effort=10 velocity=1.0 -> lower=-0.7 upper=1.57 effort=10 velocity=1.0; origin xyz=0 0 0.035 rpy=0 0 0 -> xyz=0 0 0.04 rpy=0 0 0
- joint j_f3_s1_to_f3_s2: limit lower=-0.3 upper=1.4 effort=10 velocity=1.0 -> lower=-0.7 upper=1.57 effort=10 velocity=1.0; origin xyz=0 0 0.06 rpy=0 0 0 -> xyz=0 0 0.05 rpy=0 0 0
- joint j_f3_s2_to_f3_s3: limit lower=-0.3 upper=1.4 effort=10 velocity=1.0 -> lower=-0.7 upper=1.57 effort=10 velocity=1.0
- joint j_f4_s1_to_f4_s2: limit lower=-0.3 upper=1.4 effort=10 velocity=1.0 -> lower=-0.7 upper=1.57 effort=10 velocity=1.0; origin xyz=0 0 0.055 rpy=0 0 0 -> xyz=0 0 0.05 rpy=0 0 0
- joint j_f4_s2_to_f4_s3: limit lower=-0.3 upper=1.4 effort=10 velocity=1.0 -> lower=-0.7 upper=1.57 effort=10 velocity=1.0; origin xyz=0 0 0.035 rpy=0 0 0 -> xyz=0 0 0.04 rpy=0 0 0

Commit message: chore: fix scene config

File: generated/robot.urdf (robot description, URDF)
Before this commit: robot pydantic_robot, 13 links, 12 joints
Links:
- added link fingertipf1, mass 0.01; collision sphere radius=0.008; visual sphere radius=0.008
- added link fingertipf2, mass 0.01; collision sphere radius=0.008; visual sphere radius=0.008
- added link fingertipf3, mass 0.01; collision sphere radius=0.008; visual sphere radius=0.008
- added link fingertipf4, mass 0.01; collision sphere radius=0.008; visual sphere radius=0.008
Joints:
- added joint j_f1_s3_to_fingertipf1: type fixed, parent f1_s3, child fingertipf1, origin xyz=0 0 0.03 rpy=0 0 0
- added joint j_f2_s3_to_fingertipf2: type fixed, parent f2_s3, child fingertipf2, origin xyz=0 0 0.03 rpy=0 0 0
- added joint j_f3_s3_to_fingertipf3: type fixed, parent f3_s3, child fingertipf3, origin xyz=0 0 0.03 rpy=0 0 0
- added joint j_f4_s3_to_fingertipf4: type fixed, parent f4_s3, child fingertipf4, origin xyz=0 0 0.03 rpy=0 0 0
